File: hypjolin.kicad_sch (KiCad schematic)
At the start: 321 parts, among them IC1 4021D, IC2 TL074, IC3 SSI2164, IC4 TL072, IC5 TL074, IC6 TL074, IC7 LM78L09, IC8 LM79L09, IC9 TL072, J1 freq_cv_in_a, J10 run_cv, J11 xor, J12 freq_cv_in_filter, J13 CONN_4_M, J14 Limiter_Bypass, J15 out -U, J16 out U, J17 out Z, J18 out -Z, J19 out Y, J2 freq_cv_in_b, J20 out -Y, J21 out -X, J22 out X, J23 gain_mod, J24 rate_mod, J25 damp_mod, J26 banana gnd, J27 chassis gnd, J28 DC+_From_Brick, J29 GND_From_Brick, J3 ext_in, J30 Conn_01x04_Male, J31 CONN_4_P, J32 CONN_5_M, J33 CONN_5_P, J34 CONN_2_M, J35 CONN_2_P, J36 CONN_6_M, J37 CONN_6_P, J38 CONN_1_M, J39 CONN_1_P, J4 p2, J40 CONN_3_P, J41 CONN_3_M, J5 t1, J6 t2, J7 p1, J8 out_amp, J9 pwm, Q1 3904, Q2 BC857, Q3 BC847, Q4 BC857, Q5 BC857, SW1 SUBMINI_SPDT, SW2 SUBMINI_SPDT, U1 LM13700, U2 LM13700, U3 TL074, U4 TL074, U5 LM13700, U6 TL074, U7 TL074, U8 TL074, U9 DJ06D2412A

Commit message: cleanup / fixes
Parts:
- J26: value banana gnd -> Banana GND
- J27: value chassis gnd -> Chassis GND
- J28: value DC+_From_Brick -> Brick DC+
- J29: value GND_From_Brick -> Brick GND
- SW1, SW2: footprint Connector_Triglav:SW_Toggle_Blue_wSlots -> Connector_Triglav:1082MS1T1B1M2QEEVX
Changed lines of the file:
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@@
       (effects (font (size 1.143 1.143)) (justify right))
     )
-    (property "Footprint" "Connector_Triglav:SW_Toggle_Blue_wSlots" (id 2) (at 803.402 767.08 0)
+    (property "Footprint" "Connector_Triglav:1082MS1T1B1M2QEEVX" (id 2) (at 803.402 767.08 0)
       (effects (font (size 0.508 0.508)) hide)
     )
@@
     (in_bom yes) (on_board yes)
     (property "Reference" "J28" (id 0) (at 84.455 709.93 0))
-    (property "Value" "DC+_From_Brick" (id 1) (at 74.93 715.01 0))
+    (property "Value" "Brick DC+" (id 1) (at 78.74 715.01 0))
     (property "Footprint" "Connector_Pin:Pin_D1.4mm_L8.5mm_W2.8mm_FlatFork" (id 2) (at 83.82 715.01 0)
       (effects (font (size 1.27 1.27)) hide)
@@
     (in_bom yes) (on_board yes)
     (property "Reference" "J27" (id 0) (at 84.455 707.39 0))
-    (property "Value" "chassis gnd" (id 1) (at 77.47 712.47 0))
+    (property "Value" "Chassis GND" (id 1) (at 77.47 712.47 0))
     (property "Footprint" "Connector_Pin:Pin_D1.4mm_L8.5mm_W2.8mm_FlatFork" (id 2) (at 83.82 712.47 0)
       (effects (font (size 1.27 1.27)) hide)
@@
     (in_bom yes) (on_board yes)
     (property "Reference" "J29" (id 0) (at 84.455 712.47 0))
-    (property "Value" "GND_From_Brick" (id 1) (at 74.93 717.55 0))
+    (property "Value" "Brick GND" (id 1) (at 78.74 717.55 0))
     (property "Footprint" "Connector_Pin:Pin_D1.4mm_L8.5mm_W2.8mm_FlatFork" (id 2) (at 83.82 717.55 0)
       (effects (font (size 1.27 1.27)) hide)
@@
     (in_bom yes) (on_board yes)
     (property "Reference" "J26" (id 0) (at 84.455 704.85 0))
-    (property "Value" "banana gnd" (id 1) (at 77.47 709.93 0))
+    (property "Value" "Banana GND" (id 1) (at 77.47 709.93 0))
     (property "Footprint" "Connector_Pin:Pin_D1.4mm_L8.5mm_W2.8mm_FlatFork" (id 2) (at 83.82 709.93 0)
       (effects (font (size 1.27 1.27)) hide)
@@
       (effects (font (size 1.143 1.143)))
     )
-    (property "Footprint" "Connector_Triglav:SW_Toggle_Blue_wSlots" (id 2) (at 694.182 113.03 0)
+    (property "Footprint" "Connector_Triglav:1082MS1T1B1M2QEEVX" (id 2) (at 694.182 113.03 0)
       (effects (font (size 0.508 0.508)) hide)
     )
@@
     )
     (pin "1")
-    (pin "3")
     (pin "2")
+    (pin "3")
   )
   (symbol (lib_id "Amplifier_Operational:LM13700") (at 312.42 753.11 0) (unit 2)
@@
     )
     (path "/e5e6824a-6a09-4d15-9dd5-4484c3234bc3"
-      (reference "J26") (unit 1) (value "banana gnd") (footprint "Connector_Pin:Pin_D1.4mm_L8.5mm_W2.8mm_FlatFork")
+      (reference "J26") (unit 1) (value "Banana GND") (footprint "Connector_Pin:Pin_D1.4mm_L8.5mm_W2.8mm_FlatFork")
     )
     (path "/7da7cba4-c13c-4ea2-91cf-d75ca9e56ff0"
-      (reference "J27") (unit 1) (value "chassis gnd") (footprint "Connector_Pin:Pin_D1.4mm_L8.5mm_W2.8mm_FlatFork")
+      (reference "J27") (unit 1) (value "Chassis GND") (footprint "Connector_Pin:Pin_D1.4mm_L8.5mm_W2.8mm_FlatFork")
     )
     (path "/7c260da1-b4dc-4bae-b853-3b0996128cf0"
-      (reference "J28") (unit 1) (value "DC+_From_Brick") (footprint "Connector_Pin:Pin_D1.4mm_L8.5mm_W2.8mm_FlatFork")
+      (reference "J28") (unit 1) (value "Brick DC+") (footprint "Connector_Pin:Pin_D1.4mm_L8.5mm_W2.8mm_FlatFork")
     )
     (path "/dd6f8ec3-1220-434b-9dce-422ffdf6fbed"
-      (reference "J29") (unit 1) (value "GND_From_Brick") (footprint "Connector_Pin:Pin_D1.4mm_L8.5mm_W2.8mm_FlatFork")
+      (reference "J29") (unit 1) (value "Brick GND") (footprint "Connector_Pin:Pin_D1.4mm_L8.5mm_W2.8mm_FlatFork")
     )
     (path "/f6218624-f97f-42da-a48e-de117c7d6db2"
@@
     )
     (path "/edca8aa6-bac9-4e18-9ef7-051cbe8f4677"
-      (reference "SW1") (unit 1) (value "SUBMINI_SPDT") (footprint "Connector_Triglav:SW_Toggle_Blue_wSlots")
+      (reference "SW1") (unit 1) (value "SUBMINI_SPDT") (footprint "Connector_Triglav:1082MS1T1B1M2QEEVX")
     )
     (path "/2ed92152-95a9-4f5d-9ba9-66d02abaebc0"
-      (reference "SW2") (unit 1) (value "SUBMINI_SPDT") (footprint "Connector_Triglav:SW_Toggle_Blue_wSlots")
+      (reference "SW2") (unit 1) (value "SUBMINI_SPDT") (footprint "Connector_Triglav:1082MS1T1B1M2QEEVX")
     )
     (path "/bded9836-83aa-472e-b557-90a8d914a485"

Commit message: -
Parts:
- C15, C16, C33, C34: value 22µ -> 22u; Manufacturer_Part_Number EEE-FN1A470UR -> EEEFN1C220R
Changed lines of the file:
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@@
     (in_bom yes) (on_board yes)
     (property "Reference" "C15" (id 0) (at 188.3918 306.07 0))
-    (property "Value" "22µ" (id 1) (at 186.0804 306.07 0))
+    (property "Value" "22u" (id 1) (at 186.0804 306.07 0))
     (property "Footprint" "Akiyuki:CAPAE430X610N" (id 2) (at 182.88 308.61 0)
       (effects (font (size 1.27 1.27)) (justify left) hide)
@@
       (effects (font (size 1.27 1.27)) (justify left) hide)
     )
-    (property "Manufacturer_Part_Number" "EEE-FN1A470UR" (id 7) (at 170.18 308.61 0)
+    (property "Manufacturer_Part_Number" "EEEFN1C220R" (id 7) (at 170.18 308.61 0)
       (effects (font (size 1.27 1.27)) (justify left) hide)
     )
@@
     (in_bom yes) (on_board yes)
     (property "Reference" "C16" (id 0) (at 188.3918 318.77 0))
-    (property "Value" "22µ" (id 1) (at 186.0804 318.77 0))
+    (property "Value" "22u" (id 1) (at 186.0804 318.77 0))
     (property "Footprint" "Akiyuki:CAPAE430X610N" (id 2) (at 182.88 321.31 0)
       (effects (font (size 1.27 1.27)) (justify left) hide)
@@
       (effects (font (size 1.27 1.27)) (justify left) hide)
     )
-    (property "Manufacturer_Part_Number" "EEE-FN1A470UR" (id 7) (at 170.18 321.31 0)
+    (property "Manufacturer_Part_Number" "EEEFN1C220R" (id 7) (at 170.18 321.31 0)
       (effects (font (size 1.27 1.27)) (justify left) hide)
     )
@@
     (in_bom yes) (on_board yes)
     (property "Reference" "C33" (id 0) (at 152.8318 374.65 0))
-    (property "Value" "22µ" (id 1) (at 150.5204 374.65 0))
+    (property "Value" "22u" (id 1) (at 150.5204 374.65 0))
     (property "Footprint" "Akiyuki:CAPAE430X610N" (id 2) (at 147.32 377.19 0)
       (effects (font (size 1.27 1.27)) (justify left) hide)
@@
       (effects (font (size 1.27 1.27)) (justify left) hide)
     )
-    (property "Manufacturer_Part_Number" "EEE-FN1A470UR" (id 7) (at 134.62 377.19 0)
+    (property "Manufacturer_Part_Number" "EEEFN1C220R" (id 7) (at 134.62 377.19 0)
       (effects (font (size 1.27 1.27)) (justify left) hide)
     )
@@
     (in_bom yes) (on_board yes)
     (property "Reference" "C34" (id 0) (at 152.8318 387.35 0))
-    (property "Value" "22µ" (id 1) (at 150.5204 387.35 0))
+    (property "Value" "22u" (id 1) (at 150.5204 387.35 0))
     (property "Footprint" "Akiyuki:CAPAE430X610N" (id 2) (at 147.32 389.89 0)
       (effects (font (size 1.27 1.27)) (justify left) hide)
@@
       (effects (font (size 1.27 1.27)) (justify left) hide)
     )
-    (property "Manufacturer_Part_Number" "EEE-FN1A470UR" (id 7) (at 134.62 389.89 0)
+    (property "Manufacturer_Part_Number" "EEEFN1C220R" (id 7) (at 134.62 389.89 0)
       (effects (font (size 1.27 1.27)) (justify left) hide)
     )
@@
     )
     (path "/434d14e5-f905-42af-94ce-e595f5ed3563"
-      (reference "C15") (unit 1) (value "22µ") (footprint "Akiyuki:CAPAE430X610N")
+      (reference "C15") (unit 1) (value "22u") (footprint "Akiyuki:CAPAE430X610N")
     )
     (path "/701b70cb-ded2-40b1-a13d-f484468bd824"
-      (reference "C16") (unit 1) (value "22µ") (footprint "Akiyuki:CAPAE430X610N")
+      (reference "C16") (unit 1) (value "22u") (footprint "Akiyuki:CAPAE430X610N")
     )
     (path "/695b4930-a2b9-444e-8d0a-1bf312d55acc"
@@
     )
     (path "/d1083f0e-8328-451b-9aa5-a3baa390152f"
-      (reference "C33") (unit 1) (value "22µ") (footprint "Akiyuki:CAPAE430X610N")
+      (reference "C33") (unit 1) (value "22u") (footprint "Akiyuki:CAPAE430X610N")
     )
     (path "/e9cf5724-b659-4c95-880c-ce4b5c794469"
-      (reference "C34") (unit 1) (value "22µ") (footprint "Akiyuki:CAPAE430X610N")
+      (reference "C34") (unit 1) (value "22u") (footprint "Akiyuki:CAPAE430X610N")
     )
     (path "/70847bd2-29fb-4160-ab48-adb8706abc35"

Commit message: silkscreen fixes
Parts:
- J14: value Limiter_Bypass -> Limiter
Changed lines of the file:
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@@
       (effects (font (size 1.27 1.27)) (justify right))
     )
-    (property "Value" "Limiter_Bypass" (id 1) (at 588.01 560.0699 0)
+    (property "Value" "Limiter" (id 1) (at 588.01 560.0699 0)
       (effects (font (size 1.27 1.27)) (justify right))
     )
@@
     )
     (path "/b18475d5-6343-4acb-bd24-25e10771e259"
-      (reference "J14") (unit 1) (value "Limiter_Bypass") (footprint "Connector_PinHeader_2.54mm:PinHeader_1x02_P2.54mm_Vertical")
+      (reference "J14") (unit 1) (value "Limiter") (footprint "Connector_PinHeader_2.54mm:PinHeader_1x02_P2.54mm_Vertical")
     )
     (path "/546c834a-8fe9-4bc4-8620-035838b0cfd9"

Commit message: track cleanup, 3D model update
Parts:
- U9: footprint Connector_B:DIP1549W45P254L3404H940Q24 -> Package_DIP:DIP-24_W15.24mm
Changed lines of the file:
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@@
       (effects (font (size 1.27 1.27)) (justify left))
     )
-    (property "Footprint" "Connector_B:DIP1549W45P254L3404H940Q24" (id 2) (at 102.87 669.29 0)
+    (property "Footprint" "Package_DIP:DIP-24_W15.24mm" (id 2) (at 102.87 669.29 0)
       (effects (font (size 1.27 1.27)) hide)
     )
@@
     )
     (path "/bf0bffb0-76aa-41c5-979d-ca96c48f2290"
-      (reference "U9") (unit 1) (value "DJ06D2412A") (footprint "Connector_B:DIP1549W45P254L3404H940Q24")
+      (reference "U9") (unit 1) (value "DJ06D2412A") (footprint "Package_DIP:DIP-24_W15.24mm")
     )
     (path "/d14e205e-53df-4f30-bedb-f4b3bb3c1818"

Commit message: board fixes
Parts:
- removed D33: 1N5819HW-7-F, digikey-footprints:SOD-123, symbol dk_Diodes-Rectifiers-Single:1N5819HW-7-F
- added D33: 1N5819WS, Triglav:D_SOD-323, symbol voltage_processor-rescue:1N5819-Diode
- D12, D13: value 1N5819 -> 1N5819WS; footprint Triglav:D_SOD-123 -> Triglav:D_SOD-323
- D14, D15, D16, D17, D18, D19, D20, D21, D22, D23, D24, D25, D26: footprint Diode_SMD:D_SOD-123 -> Triglav:D_SOD-123
- U1, U2, U5: footprint Package_SO:SOIC-16_3.9x9.9mm_P1.27mm -> Triglav:SO-16_3.9x9.9mm_P1.27mm
- U3, U4, U6, U7, U8: footprint Package_SO:SOIC-14_3.9x8.7mm_P1.27mm -> Triglav:SO-14_3.9x8.65mm_P1.27mm
Connections:
- net GND: now also J13.1 (Pin_1), J13.2 (Pin_2), J32.10 (Pin_10)
- net P / GND: now also J31.1 (Pin_1), J31.2 (Pin_2), J33.10 (Pin_10)
- net P / damp_mod: no longer J33.10 (Pin_10)
- net P / gain_mod: no longer J31.2 (Pin_2)
- net P / rate_mod: no longer J31.1 (Pin_1)
- net damp_mod: no longer J32.10 (Pin_10)
- net gain_mod: no longer J13.2 (Pin_2)
- net rate_mod: no longer J13.1 (Pin_1)
- net at F1.2, U9.22 (+Vin), U9.23 (+Vin): now also D33.1 (K)
- net at J29.1 (Pin_1), U9.2 (-Vin), U9.3 (-Vin): now also D33.2 (A)
Other:
- moved on the sheet: J12, J23, J24, J25

Commit message: first prototype
Parts:
- D10, D7, D8, D9: value 1N4004 -> 1N4004W
Changed lines of the file:
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@@
     (in_bom yes) (on_board yes) (fields_autoplaced)
     (property "Reference" "D7" (id 0) (at 144.78 328.93 0))
-    (property "Value" "1N4004" (id 1) (at 144.78 331.47 0))
+    (property "Value" "1N4004W" (id 1) (at 144.78 331.47 0))
     (property "Footprint" "Triglav:D_SOD-123" (id 2) (at 144.78 330.835 0)
       (effects (font (size 1.27 1.27)) hide)
@@
       (effects (font (size 1.27 1.27)) (justify left))
     )
-    (property "Value" "1N4004" (id 1) (at 163.195 307.3399 90)
+    (property "Value" "1N4004W" (id 1) (at 163.195 307.3399 90)
       (effects (font (size 1.27 1.27)) (justify left))
     )
@@
       (effects (font (size 1.27 1.27)) (justify left))
     )
-    (property "Value" "1N4004" (id 1) (at 163.195 320.0399 90)
+    (property "Value" "1N4004W" (id 1) (at 163.195 320.0399 90)
       (effects (font (size 1.27 1.27)) (justify left))
     )
@@
     (in_bom yes) (on_board yes) (fields_autoplaced)
     (property "Reference" "D8" (id 0) (at 144.78 283.21 0))
-    (property "Value" "1N4004" (id 1) (at 144.78 285.75 0))
+    (property "Value" "1N4004W" (id 1) (at 144.78 285.75 0))
     (property "Footprint" "Triglav:D_SOD-123" (id 2) (at 144.78 294.005 0)
       (effects (font (size 1.27 1.27)) hide)
@@
     )
     (path "/45532785-bae6-4b1c-8e24-5737af8d9aed"
-      (reference "D7") (unit 1) (value "1N4004") (footprint "Triglav:D_SOD-123")
+      (reference "D7") (unit 1) (value "1N4004W") (footprint "Triglav:D_SOD-123")
     )
     (path "/c318e0a7-0443-460b-9f50-40032cf6db4c"
-      (reference "D8") (unit 1) (value "1N4004") (footprint "Triglav:D_SOD-123")
+      (reference "D8") (unit 1) (value "1N4004W") (footprint "Triglav:D_SOD-123")
     )
     (path "/83b30b86-fd50-4628-a182-55b23bdab511"
-      (reference "D9") (unit 1) (value "1N4004") (footprint "Triglav:D_SOD-123")
+      (reference "D9") (unit 1) (value "1N4004W") (footprint "Triglav:D_SOD-123")
     )
     (path "/90d6ac8a-e6d6-47b5-80d7-e0ac1a5fef9e"
-      (reference "D10") (unit 1) (value "1N4004") (footprint "Triglav:D_SOD-123")
+      (reference "D10") (unit 1) (value "1N4004W") (footprint "Triglav:D_SOD-123")
     )
     (path "/7ebd524e-abc2-46ff-8d8f-8171936b36b6"

Commit message: Rev.2
Fix issues with rev.1, add TT version
Parts:
- removed D11: 1N5819*, Triglav:D_SOD-123, symbol voltage_processor-rescue:1N5819-Diode
- added J42: Jack GND, Connector_Pin:Pin_D1.4mm_L8.5mm_W2.8mm_FlatFork, symbol Connector:Conn_01x01_Female
- Q2, Q4, Q5: value BC857 -> 3906
- Q3: value BC847 -> 3904
- R117, R133, R142, R147: value RLED -> 1k
Connections:
- net GND: now also J42.1 (Pin_1); no longer J32.1 (Pin_1)
- net P / GND: now also rate1.3 (E); no longer J33.1 (Pin_1), rate1.1 (A)
- net P / VCC: no longer rate1.3 (E)
- net VEE: now also J32.1 (Pin_1)
- new net P / VEE: J33.1 (Pin_1), rate1.1 (A)
Other:
- moved on the sheet: R52, R53

Commit message: Cleanup
Parts:
- C32: value 33p -> 100p
- R66: value 20k -> 4k7
Other:
- moved on the sheet: C32, R78
