File: hypjolin.kicad_sch (KiCad schematic)
At the start: 321 parts, among them IC1 4021D, IC2 TL074, IC3 SSI2164, IC4 TL072, IC5 TL074, IC6 TL074, IC7 LM78L09, IC8 LM79L09, IC9 TL072, J1 freq_cv_in_a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

Commit message: Cleanup
Other:
- moved on the sheet: C11, C12, C13, C14, C15, C16, C17, C18, C19, C20, C21, C22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

Commit message: Cleaned up panel graphics file
Other:
- note added: "HYP"
- note added: "JOLIN"
- note added: "PCB INTERCONNECT"
- note added: "POWER"
- moved on the sheet: C1, C10, C11, C12, C13, C14, C15, C16, C17, C18, C19, C2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
